File: MP1584-tryout.sch (KiCad schematic (older format))
At the start: 15 parts, among them J1 Conn_01x03_Female, U1 MP1584

Commit message: final,
Parts:
- L1: footprint footprint-lib:L_SMD_ALL -> w_smd_inductors:inductor_smd_6.8x3.8mm
- U1: footprint footprint-lib:MP2303,SOIC-8_3.9x4.9mm_P1.27mm,thermal_via -> footprint-lib:MP1584,SOIC-8_3.9x4.9mm_P1.27mm,thermal_via
Changed lines of the file:
@@
 EESchema Schematic File Version 4
+LIBS:MP1584-tryout-cache
 EELAYER 29 0
 EELAYER END
@@
 F 0 "U1" H 5800 4050 50  0000 C CNN
 F 1 "MP1584" H 5800 3950 50  0000 C CNN
-F 2 "footprint-lib:MP2303,SOIC-8_3.9x4.9mm_P1.27mm,thermal_via" H 5800 2500 50  0001 C CNN
+F 2 "footprint-lib:MP1584,SOIC-8_3.9x4.9mm_P1.27mm,thermal_via" H 5800 2500 50  0001 C CNN
 F 3 "" H 5800 3350 50  0001 C CNN
 	1    5800 3350
@@
 F 0 "L1" V 7750 3200 50  0000 C CNN
 F 1 "L_15uH" V 7650 3200 50  0000 C CNN
-F 2 "footprint-lib:L_SMD_ALL" H 7550 3200 50  0001 C CNN
+F 2 "w_smd_inductors:inductor_smd_6.8x3.8mm" H 7550 3200 50  0001 C CNN
 F 3 "test_datasheet" H 7550 3200 50  0001 C CNN
 	1    7550 3200

Commit message: update,
Parts:
- C1: value C104,0603 -> C104,0805; footprint Capacitor_SMD:C_0603_1608Metric_Pad1.05x0.95mm_HandSolder -> Resistor_SMD:R_0805_2012Metric
- C3: value C151,0603 -> C151,0805; footprint Capacitor_SMD:C_0603_1608Metric_Pad1.05x0.95mm_HandSolder -> Capacitor_SMD:C_0805_2012Metric
- R1, R4, R6: value R104,0603 -> R104,0805; footprint Resistor_SMD:R_0603_1608Metric_Pad1.05x0.95mm_HandSolder -> Resistor_SMD:R_0805_2012Metric
- R2: value R224,0603 -> R224,0805; footprint Resistor_SMD:R_0603_1608Metric_Pad1.05x0.95mm_HandSolder -> Resistor_SMD:R_0805_2012Metric
- R3: value R240,0603 -> R240,0805; footprint Resistor_SMD:R_0603_1608Metric_Pad1.05x0.95mm_HandSolder -> Resistor_SMD:R_0805_2012Metric
- R5: value R433,0603 -> R433,0805; footprint Resistor_SMD:R_0603_1608Metric_Pad1.05x0.95mm_HandSolder -> Resistor_SMD:R_0805_2012Metric
Connections:
- net SW_OUT: now reaches C1.1, D1.1 (K), L1.1, U1.1 (SW)
Other:
- note added: "Features:\n\n- Module type: Non-isolated step-down module (buck) ;\n- Input voltage: 7~28VDC;\n- Output voltage: 5VDC+/-3%;\n- No load current: small, 2mA;\n- Output Current: 2.5A (MAX) ;\n- Continuous current: 1A (MAX) ;\n- Conversion efficiency: 92% (MAX) ;\n- Switching Frequency: 1MHz typical.\n"
- moved on the sheet: D1
